File: conductive/conductive.sch (KiCad schematic (older format))
At the start: 14 parts, among them U1 AD8534, U2 AD8531

Commit message: update
Parts:
- added C1, C2: C, symbol C
- added J1: Conn_01x08, symbol Conn_01x08
- added J2: Screw_Terminal_01x02, symbol Screw_Terminal_01x02
- added R4B, R4B? (x6): R, symbol R
- added U1: TLE2426, symbol TLE2426
- added U2: 74H4051, symbol 74H4051
- gave numbers to parts that had none: 1
- renumbered R4 to R4A, U1 to U3, U2 to U4
Connections:
- net +3V3: now also C2.2, J1.1 (Pin_1), U1.3 (IN), U2.16 (VCC)
- net GND: now also C1.1, C2.1, J1.2 (Pin_2), U1.2 (COMMON), U1.4 (NC), U1.5 (NC), U1.6 (NC), U1.7 (NC), U2.7 (VEE), U2.8 (GND)
- net GNDREF: now also U1.1 (OUT)
- net PROBE_A: now also J2.1 (Pin_1)
- net PROBE_B: now also J2.2 (Pin_2), U2.3 (Z); no longer R4A.2
- net SIG_IN: now also J1.3 (Pin_3)
- net SIG_OUT: now also J1.4 (Pin_4)
- net at R5.1, U3.7 (OUT_B): now also R4A.2, R4B.2, R4B?.2, R4B?.2, R4B?.2, R4B?.2, R4B?.2, R4B?.2; no longer R4A.1
- new net: C1.2, U1.8 (NOISE_RED)
- new net S0: J1.6 (Pin_6), U2.11 (S0)
- new net S1: J1.7 (Pin_7), U2.10 (S1)
- new net S2: J1.8 (Pin_8), U2.9 (S2)
- new net Y0: R4A.1, U2.13 (Y0)
- new net Y1: R4B.1, U2.14 (Y1)
- new net Y2: R4B?.1, U2.15 (Y2)
- new net Y3: R4B?.1, U2.12 (Y3)
- new net Y4: R4B?.1, U2.1 (Y4)
- new net Y5: R4B?.1, U2.5 (Y5)
- new net Y6: R4B?.1, U2.2 (Y6)
- new net Y7: R4B?.1, U2.4 (Y7)
- new net ~E: J1.5 (Pin_5), U2.6 (~E)
Other:
- moved on the sheet: C3, D?, R1, R10, R2, R4A, R5, R6, R7, R8, R9, U3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

Commit message: update
Parts:
- added J3: Conn_01x02, symbol Conn_01x02
Connections:
- net PROBE_B: now also J3.2 (Pin_2)
- net at R4A.2, R4B.2, R4B?.2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: now also J3.1 (Pin_1)
Other:
- moved on the sheet: C1, C2, U1
Changed lines of the file:
@@
 Text GLabel 5400 6850 0    60   Input ~ 0
 Y7
+$Comp
+L +3V3 #PWR?
+U 1 1 59CF344A
+P 3000 1750
+F 0 "#PWR?" H 3000 1600 50  0001 C CNN
+F 1 "+3V3" V 3015 1878 50  0000 L CNN
+F 2 "" H 3000 1750 50  0001 C CNN
+F 3 "" H 3000 1750 50  0001 C CNN
+	1    3000 1750
+	0    -1   -1   0
+$EndComp
+$Comp
+L GND #PWR?
+U 1 1 59CF360A
+P 3000 1850
+F 0 "#PWR?" H 3000 1600 50  0001 C CNN
+F 1 "GND" V 3005 1722 50  0000 R CNN
+F 2 "" H 3000 1850 50  0001 C CNN
+F 3 "" H 3000 1850 50  0001 C CNN
+	1    3000 1850
+	0    1    1    0
+$EndComp
+Text GLabel 2350 1950 0    60   Input ~ 0
+SIG_IN
+Text GLabel 2800 2050 0    60   Input ~ 0
+SIG_OUT
+$Comp
+L Conn_01x08 J1
+U 1 1 59CF40AF
+P 3200 2050
+F 0 "J1" H 3280 2042 50  0000 L CNN
+F 1 "Conn_01x08" H 3280 1951 50  0000 L CNN
+F 2 "" H 3200 2050 50  0001 C CNN
+F 3 "" H 3200 2050 50  0001 C CNN
+	1    3200 2050
+	1    0    0    -1
+$EndComp
+Text GLabel 3000 2150 0    60   Input ~ 0
+~E
+Text GLabel 2800 2250 0    60   Input ~ 0
+S0
+Text GLabel 3000 2350 0    60   Input ~ 0
+S1
+Text GLabel 2800 2450 0    60   Input ~ 0
+S2
+$Comp
+L Screw_Terminal_01x02 J2
+U 1 1 59CF455B
+P 3200 2850
+F 0 "J2" H 3280 2842 50  0000 L CNN
+F 1 "Screw_Terminal_01x02" H 3280 2751 50  0000 L CNN
+F 2 "" H 3200 2850 50  0001 C CNN
+F 3 "" H 3200 2850 50  0001 C CNN
+	1    3200 2850
+	1    0    0    -1
+$EndComp
+Text GLabel 3000 2850 0    60   Input ~ 0
+PROBE_A
+Text GLabel 2550 2950 0    60   Input ~ 0
+PROBE_B
+$Comp
+L TLE2426 U1
+U 1 1 59CF5255
+P 1750 4350
+F 0 "U1" H 1775 4887 60  0000 C CNN
+F 1 "TLE2426" H 1775 4781 60  0000 C CNN
+F 2 "" H 1650 3800 60  0001 C CNN
+F 3 "" H 1650 3800 60  0001 C CNN
+	1    1750 4350
+	1    0    0    -1
+$EndComp
+$Comp
+L GND #PWR?
+U 1 1 59CF6DE6
+P 2300 4550
+F 0 "#PWR?" H 2300 4300 50  0001 C CNN
+F 1 "GND" V 2305 4422 50  0000 R CNN
+F 2 "" H 2300 4550 50  0001 C CNN
+F 3 "" H 2300 4550 50  0001 C CNN
+	1    2300 4550
+	0    -1   -1   0
+$EndComp
+$Comp
+L GND #PWR?
+U 1 1 59CF6E55
+P 2300 4400
+F 0 "#PWR?" H 2300 4150 50  0001 C CNN
+F 1 "GND" V 2305 4272 50  0000 R CNN
+F 2 "" H 2300 4400 50  0001 C CNN
+F 3 "" H 2300 4400 50  0001 C CNN
+	1    2300 4400
+	0    -1   -1   0
+$EndComp
+$Comp
+L GND #PWR?
+U 1 1 59CF6E92
+P 2300 4250
+F 0 "#PWR?" H 2300 4000 50  0001 C CNN
+F 1 "GND" V 2305 4122 50  0000 R CNN
+F 2 "" H 2300 4250 50  0001 C CNN
+F 3 "" H 2300 4250 50  0001 C CNN
+	1    2300 4250
+	0    -1   -1   0
+$EndComp
+$Comp
+L GND #PWR?
+U 1 1 59CF6F65
+P 1250 4550
+F 0 "#PWR?" H 1250 4300 50  0001 C CNN
+F 1 "GND" V 1255 4422 50  0000 R CNN
+F 2 "" H 1250 4550 50  0001 C CNN
+F 3 "" H 1250 4550 50  0001 C CNN
+	1    1250 4550
+	0    1    1    0
+$EndComp
+$Comp
+L GND #PWR?
+U 1 1 59CF7038
+P 1250 4250
+F 0 "#PWR?" H 1250 4000 50  0001 C CNN
+F 1 "GND" V 1255 4122 50  0000 R CNN
+F 2 "" H 1250 4250 50  0001 C CNN
+F 3 "" H 1250 4250 50  0001 C CNN
+	1    1250 4250
+	0    1    1    0
+$EndComp
+$Comp
+L GNDREF #PWR?
+U 1 1 59CF72FF
+P 1250 4100
+F 0 "#PWR?" H 1250 3850 50  0001 C CNN
+F 1 "GNDREF" V 1255 3972 50  0000 R CNN
+F 2 "" H 1250 4100 50  0001 C CNN
+F 3 "" H 1250 4100 50  0001 C CNN
+	1    1250 4100
+	0    1    1    0
+$EndComp
+$Comp
+L +3V3 #PWR?
+U 1 1 59CF776F
+P 1250 4400
+F 0 "#PWR?" H 1250 4250 50  0001 C CNN
+F 1 "+3V3" V 1265 4528 50  0000 L CNN
+F 2 "" H 1250 4400 50  0001 C CNN
+F 3 "" H 1250 4400 50  0001 C CNN
+	1    1250 4400
+	0    -1   -1   0
+$EndComp
+$Comp
+L C C1
+U 1 1 59CF7CC0
+P 2700 4100
+F 0 "C1" V 2448 4100 50  0000 C CNN
+F 1 "C" V 2539 4100 50  0000 C CNN
+F 2 "" H 2738 3950 50  0001 C CNN
+F 3 "" H 2700 4100 50  0001 C CNN
+	1    2700 4100
+	0    1    1    0
+$EndComp
+$Comp
+L GND #PWR?
+U 1 1 59CF7E61
+P 2850 4300
+F 0 "#PWR?" H 2850 4050 50  0001 C CNN
+F 1 "GND" H 2855 4127 50  0000 C CNN
+F 2 "" H 2850 4300 50  0001 C CNN
+F 3 "" H 2850 4300 50  0001 C CNN
+	1    2850 4300
+	1    0    0    -1
+$EndComp
+$Comp
+L GND #PWR?
+U 1 1 59CF812A
+P 1800 5600
+F 0 "#PWR?" H 1800 5350 50  0001 C CNN
+F 1 "GND" H 1805 5427 50  0000 C CNN
+F 2 "" H 1800 5600 50  0001 C CNN
+F 3 "" H 1800 5600 50  0001 C CNN
+	1    1800 5600
+	1    0    0    -1
+$EndComp
+$Comp
+L +3V3 #PWR?
+U 1 1 59CF8183
+P 1800 5300
+F 0 "#PWR?" H 1800 5150 50  0001 C CNN
+F 1 "+3V3" H 1815 5473 50  0000 C CNN
+F 2 "" H 1800 5300 50  0001 C CNN
+F 3 "" H 1800 5300 50  0001 C CNN
+	1    1800 5300
+	1    0    0    -1
+$EndComp
+$Comp
+L C C2
+U 1 1 59CF81DC
+P 1800 5450
+F 0 "C2" H 1685 5404 50  0000 R CNN
+F 1 "C" H 1685 5495 50  0000 R CNN
+F 2 "" H 1838 5300 50  0001 C CNN
+F 3 "" H 1800 5450 50  0001 C CNN
+	1    1800 5450
+	-1   0    0    1
+$EndComp
 Wire Wire Line
 	6300 3200 6850 3200
@@
 	6600 4350 6600 3950
 Connection ~ 6600 3950
-$Comp
-L +3V3 #PWR?
-U 1 1 59CF344A
-P 3000 1750
-F 0 "#PWR?" H 3000 1600 50  0001 C CNN
-F 1 "+3V3" V 3015 1878 50  0000 L CNN
-F 2 "" H 3000 1750 50  0001 C CNN
-F 3 "" H 3000 1750 50  0001 C CNN
-	1    3000 1750
-	0    -1   -1   0
-$EndComp
-$Comp
-L GND #PWR?
-U 1 1 59CF360A
-P 3000 1850
-F 0 "#PWR?" H 3000 1600 50  0001 C CNN
-F 1 "GND" V 3005 1722 50  0000 R CNN
-F 2 "" H 3000 1850 50  0001 C CNN
-F 3 "" H 3000 1850 50  0001 C CNN
-	1    3000 1850
-	0    1    1    0
-$EndComp
-Text GLabel 2350 1950 0    60   Input ~ 0
-SIG_IN
-Text GLabel 2800 2050 0    60   Input ~ 0
-SIG_OUT
-$Comp
-L Conn_01x08 J1
-U 1 1 59CF40AF
-P 3200 2050
-F 0 "J1" H 3280 2042 50  0000 L CNN
-F 1 "Conn_01x08" H 3280 1951 50  0000 L CNN
-F 2 "" H 3200 2050 50  0001 C CNN
-F 3 "" H 3200 2050 50  0001 C CNN
-	1    3200 2050
-	1    0    0    -1
-$EndComp
-Text GLabel 3000 2150 0    60   Input ~ 0
-~E
 Wire Wire Line
 	2350 1950 3000 1950
@@
 Wire Wire Line
 	3000 2250 2800 2250
-Text GLabel 2800 2250 0    60   Input ~ 0
-S0
-Text GLabel 3000 2350 0    60   Input ~ 0
-S1
-Text GLabel 2800 2450 0    60   Input ~ 0
-S2
 Wire Wire Line
 	2800 2450 3000 2450
-$Comp
-L Screw_Terminal_01x02 J2
-U 1 1 59CF455B
-P 3200 2850
-F 0 "J2" H 3280 2842 50  0000 L CNN
-F 1 "Screw_Terminal_01x02" H 3280 2751 50  0000 L CNN
-F 2 "" H 3200 2850 50  0001 C CNN
-F 3 "" H 3200 2850 50  0001 C CNN
-	1    3200 2850
-	1    0    0    -1
-$EndComp
-Text GLabel 3000 2850 0    60   Input ~ 0
-PROBE_A
-Text GLabel 2550 2950 0    60   Input ~ 0
-PROBE_B
 Wire Wire Line
 	2550 2950 3000 2950
-$Comp
-L TLE2426 U1
-U 1 1 59CF5255
-P 2700 4000
-F 0 "U1" H 2725 4537 60  0000 C CNN
-F 1 "TLE2426" H 2725 4431 60  0000 C CNN
-F 2 "" H 2600 3450 60  0001 C CNN
-F 3 "" H 2600 3450 60  0001 C CNN
-	1    2700 4000
-	1    0    0    -1
-$EndComp
-$Comp
-L GND #PWR?
-U 1 1 59CF6DE6
-P 3250 4200
-F 0 "#PWR?" H 3250 3950 50  0001 C CNN
-F 1 "GND" V 3255 4072 50  0000 R CNN
-F 2 "" H 3250 4200 50  0001 C CNN
-F 3 "" H 3250 4200 50  0001 C CNN
-	1    3250 4200
-	0    -1   -1   0
-$EndComp
-$Comp
-L GND #PWR?
-U 1 1 59CF6E55
-P 3250 4050
-F 0 "#PWR?" H 3250 3800 50  0001 C CNN
-F 1 "GND" V 3255 3922 50  0000 R CNN
-F 2 "" H 3250 4050 50  0001 C CNN
-F 3 "" H 3250 4050 50  0001 C CNN
-	1    3250 4050
-	0    -1   -1   0
-$EndComp
-$Comp
-L GND #PWR?
-U 1 1 59CF6E92
-P 3250 3900
-F 0 "#PWR?" H 3250 3650 50  0001 C CNN
-F 1 "GND" V 3255 3772 50  0000 R CNN
-F 2 "" H 3250 3900 50  0001 C CNN
-F 3 "" H 3250 3900 50  0001 C CNN
-	1    3250 3900
-	0    -1   -1   0
-$EndComp
-$Comp
-L GND #PWR?
-U 1 1 59CF6F65
-P 2200 4200
-F 0 "#PWR?" H 2200 3950 50  0001 C CNN
-F 1 "GND" V 2205 4072 50  0000 R CNN
-F 2 "" H 2200 4200 50  0001 C CNN
-F 3 "" H 2200 4200 50  0001 C CNN
-	1    2200 4200
-	0    1    1    0
-$EndComp
-$Comp
-L GND #PWR?
-U 1 1 59CF7038
-P 2200 3900
-F 0 "#PWR?" H 2200 3650 50  0001 C CNN
-F 1 "GND" V 2205 3772 50  0000 R CNN
-F 2 "" H 2200 3900 50  0001 C CNN
-F 3 "" H 2200 3900 50  0001 C CNN
-	1    2200 3900
-	0    1    1    0
-$EndComp
-$Comp
-L GNDREF #PWR?
-U 1 1 59CF72FF
-P 2200 3750
-F 0 "#PWR?" H 2200 3500 50  0001 C CNN
-F 1 "GNDREF" V 2205 3622 50  0000 R CNN
-F 2 "" H 2200 3750 50  0001 C CNN
-F 3 "" H 2200 3750 50  0001 C CNN
-	1    2200 3750
-	0    1    1    0
-$EndComp
-$Comp
-L +3V3 #PWR?
-U 1 1 59CF776F
-P 2200 4050
-F 0 "#PWR?" H 2200 3900 50  0001 C CNN
-F 1 "+3V3" V 2215 4178 50  0000 L CNN
-F 2 "" H 2200 4050 50  0001 C CNN
-F 3 "" H 2200 4050 50  0001 C CNN
-	1    2200 4050
-	0    -1   -1   0
-$EndComp
-$Comp
-L C C1
-U 1 1 59CF7CC0
-P 3650 3750
-F 0 "C1" V 3398 3750 50  0000 C CNN
-F 1 "C" V 3489 3750 50  0000 C CNN
-F 2 "" H 3688 3600 50  0001 C CNN
-F 3 "" H 3650 3750 50  0001 C CNN
-	1    3650 3750
-	0    1    1    0
-$EndComp
-Wire Wire Line
-	3250 3750 3500 3750
-Wire Wire Line
-	3800 3750 3800 3950
-$Comp
-L GND #PWR?
-U 1 1 59CF7E61
-P 3800 3950
-F 0 "#PWR?" H 3800 3700 50  0001 C CNN
-F 1 "GND" H 3805 3777 50  0000 C CNN
-F 2 "" H 3800 3950 50  0001 C CNN
-F 3 "" H 3800 3950 50  0001 C CNN
-	1    3800 3950
-	1    0    0    -1
-$EndComp
-$Comp
-L GND #PWR?
-U 1 1 59CF812A
-P 1200 4100
-F 0 "#PWR?" H 1200 3850 50  0001 C CNN
-F 1 "GND" H 1205 3927 50  0000 C CNN
-F 2 "" H 1200 4100 50  0001 C CNN
-F 3 "" H 1200 4100 50  0001 C CNN
-	1    1200 4100
-	1    0    0    -1
-$EndComp
-$Comp
-L +3V3 #PWR?
-U 1 1 59CF8183
-P 1200 3800
-F 0 "#PWR?" H 1200 3650 50  0001 C CNN
-F 1 "+3V3" H 1215 3973 50  0000 C CNN
-F 2 "" H 1200 3800 50  0001 C CNN
-F 3 "" H 1200 3800 50  0001 C CNN
-	1    1200 3800
-	1    0    0    -1
-$EndComp
-$Comp
-L C C2
-U 1 1 59CF81DC
-P 1200 3950
-F 0 "C2" H 1085 3904 50  0000 R CNN
-F 1 "C" H 1085 3995 50  0000 R CNN
-F 2 "" H 1238 3800 50  0001 C CNN
-F 3 "" H 1200 3950 50  0001 C CNN
-	1    1200 3950
-	-1   0    0    1
-$EndComp
+Wire Wire Line
+	2300 4100 2550 4100
+Wire Wire Line
+	2850 4100 2850 4300
+$Comp
+L Conn_01x02 J3
+U 1 1 59CF9B0C
+P 6200 4650
+F 0 "J3" V 6073 4730 50  0000 L CNN
+F 1 "Conn_01x02" V 6164 4730 50  0000 L CNN
+F 2 "" H 6200 4650 50  0001 C CNN
+F 3 "" H 6200 4650 50  0001 C CNN
+	1    6200 4650
+	0    1    1    0
+$EndComp
+Wire Wire Line
+	6100 3800 6100 4450
+Connection ~ 6100 3800
+Wire Wire Line
+	6200 3950 6200 4450
+Connection ~ 6200 3950
 $EndSCHEMATC
