File: conductive/conductive.sch (KiCad schematic (older format))
At the start: 28 parts, among them J1 Conn_01x08, J2 Screw_Terminal_01x02, J3 Conn_01x02, U1 TLE2426, U2 74H4051, U3 AD8534, U4 AD8531

Commit message: update
Parts:
- gave numbers to parts that had none: 6
Changed lines of the file:
@@
 $EndComp
 $Comp
-L R R4B?
+L R R4C
 U 1 1 59CF0EF5
 P 5550 5100
-F 0 "R4B?" V 5757 5100 50  0000 C CNN
+F 0 "R4C" V 5757 5100 50  0000 C CNN
 F 1 "R" V 5666 5100 50  0000 C CNN
 F 2 "" V 5480 5100 50  0001 C CNN
@@
 $EndComp
 $Comp
-L R R4B?
+L R R4D
 U 1 1 59CF0F35
 P 5550 5450
-F 0 "R4B?" V 5757 5450 50  0000 C CNN
+F 0 "R4D" V 5757 5450 50  0000 C CNN
 F 1 "R" V 5666 5450 50  0000 C CNN
 F 2 "" V 5480 5450 50  0001 C CNN
@@
 $EndComp
 $Comp
-L R R4B?
+L R R4E
 U 1 1 59CF0F87
 P 5550 5800
-F 0 "R4B?" V 5757 5800 50  0000 C CNN
+F 0 "R4E" V 5757 5800 50  0000 C CNN
 F 1 "R" V 5666 5800 50  0000 C CNN
 F 2 "" V 5480 5800 50  0001 C CNN
@@
 $EndComp
 $Comp
-L R R4B?
+L R R4F
 U 1 1 59CF0FCD
 P 5550 6150
-F 0 "R4B?" V 5757 6150 50  0000 C CNN
+F 0 "R4F" V 5757 6150 50  0000 C CNN
 F 1 "R" V 5666 6150 50  0000 C CNN
 F 2 "" V 5480 6150 50  0001 C CNN
@@
 $EndComp
 $Comp
-L R R4B?
+L R R4G
 U 1 1 59CF1013
 P 5550 6500
-F 0 "R4B?" V 5757 6500 50  0000 C CNN
+F 0 "R4G" V 5757 6500 50  0000 C CNN
 F 1 "R" V 5666 6500 50  0000 C CNN
 F 2 "" V 5480 6500 50  0001 C CNN
@@
 $EndComp
 $Comp
-L R R4B?
+L R R4H
 U 1 1 59CF1070
 P 5550 6850
-F 0 "R4B?" V 5757 6850 50  0000 C CNN
+F 0 "R4H" V 5757 6850 50  0000 C CNN
 F 1 "R" V 5666 6850 50  0000 C CNN
 F 2 "" V 5480 6850 50  0001 C CNN

Commit message: update
Parts:
- added J4: Conn_01x06, symbol Conn_01x06
- gave numbers to parts that had none: 2
- renumbered R4A to R4A1, R4B to R4B1, R4C to R4C1, R4D to R4D1, R4E to R4E1, R4F to R4F1, R4G to R4G1, R4H to R4H1
Connections:
- net PROBE_A: now also J4.1 (Pin_1)
- net PROBE_B: now also J4.2 (Pin_2)
- net SIG_IN: now also J4.3 (Pin_3)
- net SIG_OUT: now also J4.6 (Pin_6)
- new net V_B: J4.4 (Pin_4)
- new net V_C: J4.5 (Pin_5)

Commit message: update
Parts:
- removed J4: Conn_01x06, symbol Conn_01x06
- added J4: Conn_01x07, Pin_Headers:Pin_Header_Straight_1x07_Pitch2.54mm, symbol Conn_01x07
- C1, C2, C3: footprint (none) -> Capacitors_SMD:C_0805
- D1, D2: footprint (none) -> Diodes_SMD:D_1206
- J1: footprint (none) -> Pin_Headers:Pin_Header_Straight_1x08_Pitch2.54mm
- J2: footprint (none) -> Connectors_Terminal_Blocks:TerminalBlock_4UCON_19963_02x3.5mm_Straight
- J3: footprint (none) -> Pin_Headers:Pin_Header_Straight_1x02_Pitch2.54mm
- R1, R10, R2, R4A1, R4B1, R4C1, R4D1, R4E1, R4F1, R4G1, R4H1, R5, R6, R7, R8, R9: footprint (none) -> Resistors_SMD:R_0805
- U1, U4: footprint (none) -> SMD_Packages:SOIC-8-N
- U2: footprint (none) -> SMD_Packages:SO-16-N
- U3: footprint (none) -> SMD_Packages:SOIC-14_N
Connections:
- net GNDREF: now also J4.7 (Pin_7)
- net PROBE_A: now also J2.2 (Pin_2), J4.2 (Pin_2); no longer J2.1 (Pin_1)
- net PROBE_B: now also J2.1 (Pin_1), J4.3 (Pin_3); no longer J2.2 (Pin_2)
- net S0: now also J1.8 (Pin_8); no longer J1.6 (Pin_6)
- net S2: now also J1.6 (Pin_6); no longer J1.8 (Pin_8)
- net SIG_IN: now also J4.1 (Pin_1)
- net SIG_OUT: now also J4.6 (Pin_6)
- net V_B: now also J3.1 (Pin_1), R4A1.2, R4B1.2, R4C1.2, R4D1.2, R4E1.2, R4F1.2, R4G1.2, R4H1.2, R5.1, U3.7 (OUT_B), J4.4 (Pin_4)
- net V_C: now also D1.1 (K), D2.2 (A), U3.8 (OUT_C), J4.5 (Pin_5)
- net at R1.1, U3.2 (-IN_A): now also R2.1
Other:
- moved on the sheet: R2
Changed lines of the file:
@@
 F 0 "U3" H 7350 2837 60  0000 C CNN
 F 1 "AD8534" H 7350 2731 60  0000 C CNN
-F 2 "" H 7300 2800 60  0001 C CNN
+F 2 "SMD_Packages:SOIC-14_N" H 7300 2800 60  0001 C CNN
 F 3 "" H 7300 2800 60  0001 C CNN
 	1    7300 2800
@@
 F 0 "R1" V 5943 3200 50  0000 C CNN
 F 1 "R" V 6034 3200 50  0000 C CNN
-F 2 "" V 6080 3200 50  0001 C CNN
+F 2 "Resistors_SMD:R_0805" V 6080 3200 50  0001 C CNN
 F 3 "" H 6150 3200 50  0001 C CNN
 	1    6150 3200
@@
 L R R2
 U 1 1 59CE9040
-P 6400 3050
-F 0 "R2" H 6330 3004 50  0000 R CNN
-F 1 "R" H 6330 3095 50  0000 R CNN
-F 2 "" V 6330 3050 50  0001 C CNN
-F 3 "" H 6400 3050 50  0001 C CNN
-	1    6400 3050
-	-1   0    0    1
+P 6700 2900
+F 0 "R2" H 6630 2854 50  0000 R CNN
+F 1 "R" H 6630 2945 50  0000 R CNN
+F 2 "Resistors_SMD:R_0805" V 6630 2900 50  0001 C CNN
+F 3 "" H 6700 2900 50  0001 C CNN
+	1    6700 2900
+	0    -1   -1   0
 $EndComp
 $Comp
@@
 F 0 "R5" V 7607 4350 50  0000 C CNN
 F 1 "R" V 7516 4350 50  0000 C CNN
-F 2 "" V 7330 4350 50  0001 C CNN
+F 2 "Resistors_SMD:R_0805" V 7330 4350 50  0001 C CNN
 F 3 "" H 7400 4350 50  0001 C CNN
 	1    7400 4350
@@
 F 0 "R4A1" V 5757 4400 50  0000 C CNN
 F 1 "R" V 5666 4400 50  0000 C CNN
-F 2 "" V 5480 4400 50  0001 C CNN
+F 2 "Resistors_SMD:R_0805" V 5480 4400 50  0001 C CNN
 F 3 "" H 5550 4400 50  0001 C CNN
 	1    5550 4400
@@
 F 0 "R6" V 8857 4050 50  0000 C CNN
 F 1 "R" V 8766 4050 50  0000 C CNN
-F 2 "" V 8580 4050 50  0001 C CNN
+F 2 "Resistors_SMD:R_0805" V 8580 4050 50  0001 C CNN
 F 3 "" H 8650 4050 50  0001 C CNN
 	1    8650 4050
@@
 F 0 "R7" V 8857 5300 50  0000 C CNN
 F 1 "R" V 8766 5300 50  0000 C CNN
-F 2 "" V 8580 5300 50  0001 C CNN
+F 2 "Resistors_SMD:R_0805" V 8580 5300 50  0001 C CNN
 F 3 "" H 8650 5300 50  0001 C CNN
 	1    8650 5300
@@
 F 0 "R8" V 9157 3200 50  0000 C CNN
 F 1 "R" V 9066 3200 50  0000 C CNN
-F 2 "" V 8880 3200 50  0001 C CNN
+F 2 "Resistors_SMD:R_0805" V 8880 3200 50  0001 C CNN
 F 3 "" H 8950 3200 50  0001 C CNN
 	1    8950 3200
@@
 F 0 "R9" V 8557 3050 50  0000 C CNN
 F 1 "R" V 8466 3050 50  0000 C CNN
-F 2 "" V 8280 3050 50  0001 C CNN
+F 2 "Resistors_SMD:R_0805" V 8280 3050 50  0001 C CNN
 F 3 "" H 8350 3050 50  0001 C CNN
 	1    8350 3050
@@
 F 0 "R10" H 7980 2354 50  0000 R CNN
 F 1 "R" H 7980 2445 50  0000 R CNN
-F 2 "" V 7980 2400 50  0001 C CNN
+F 2 "Resistors_SMD:R_0805" V 7980 2400 50  0001 C CNN
 F 3 "" H 8050 2400 50  0001 C CNN
 	1    8050 2400
@@
 F 0 "D1" V 9146 4121 50  0000 R CNN
 F 1 "D" V 9055 4121 50  0000 R CNN
-F 2 "" H 9100 4200 50  0001 C CNN
+F 2 "Diodes_SMD:D_1206" H 9100 4200 50  0001 C CNN
 F 3 "" H 9100 4200 50  0001 C CNN
 	1    9100 4200
@@
 F 0 "D2" V 9146 4871 50  0000 R CNN
 F 1 "D" V 9055 4871 50  0000 R CNN
-F 2 "" H 9100 4950 50  0001 C CNN
+F 2 "Diodes_SMD:D_1206" H 9100 4950 50  0001 C CNN
 F 3 "" H 9100 4950 50  0001 C CNN
 	1    9100 4950
@@
 F 0 "C3" V 7448 2000 50  0000 C CNN
 F 1 "C" V 7539 2000 50  0000 C CNN
-F 2 "" H 7738 1850 50  0001 C CNN
+F 2 "Capacitors_SMD:C_0805" H 7738 1850 50  0001 C CNN
 F 3 "" H 7700 2000 50  0001 C CNN
 	1    7700 2000
@@
 F 0 "U4" H 9175 1487 60  0000 C CNN
 F 1 "AD8531" H 9175 1381 60  0000 C CNN
-F 2 "" H 9200 1450 60  0001 C CNN
+F 2 "SMD_Packages:SOIC-8-N" H 9200 1450 60  0001 C CNN
 F 3 "" H 9200 1450 60  0001 C CNN
 	1    9200 1450
@@
 F 0 "U2" H 4000 7487 60  0000 C CNN
 F 1 "74H4051" H 4000 7381 60  0000 C CNN
-F 2 "" H 4000 6100 60  0001 C CNN
+F 2 "SMD_Packages:SO-16-N" H 4000 6100 60  0001 C CNN
 F 3 "" H 4000 6100 60  0001 C CNN
 	1    4000 6100
@@
 F 0 "R4B1" V 5757 4750 50  0000 C CNN
 F 1 "R" V 5666 4750 50  0000 C CNN
-F 2 "" V 5480 4750 50  0001 C CNN
+F 2 "Resistors_SMD:R_0805" V 5480 4750 50  0001 C CNN
 F 3 "" H 5550 4750 50  0001 C CNN
 	1    5550 4750
@@
 F 0 "R4C1" V 5757 5100 50  0000 C CNN
 F 1 "R" V 5666 5100 50  0000 C CNN
-F 2 "" V 5480 5100 50  0001 C CNN
+F 2 "Resistors_SMD:R_0805" V 5480 5100 50  0001 C CNN
 F 3 "" H 5550 5100 50  0001 C CNN
 	1    5550 5100
@@
 F 0 "R4D1" V 5757 5450 50  0000 C CNN
 F 1 "R" V 5666 5450 50  0000 C CNN
-F 2 "" V 5480 5450 50  0001 C CNN
+F 2 "Resistors_SMD:R_0805" V 5480 5450 50  0001 C CNN
 F 3 "" H 5550 5450 50  0001 C CNN
 	1    5550 5450
@@
 F 0 "R4E1" V 5757 5800 50  0000 C CNN
 F 1 "R" V 5666 5800 50  0000 C CNN
-F 2 "" V 5480 5800 50  0001 C CNN
+F 2 "Resistors_SMD:R_0805" V 5480 5800 50  0001 C CNN
 F 3 "" H 5550 5800 50  0001 C CNN
 	1    5550 5800
@@
 F 0 "R4F1" V 5757 6150 50  0000 C CNN
 F 1 "R" V 5666 6150 50  0000 C CNN
-F 2 "" V 5480 6150 50  0001 C CNN
+F 2 "Resistors_SMD:R_0805" V 5480 6150 50  0001 C CNN
 F 3 "" H 5550 6150 50  0001 C CNN
 	1    5550 6150
@@
 F 0 "R4G1" V 5757 6500 50  0000 C CNN
 F 1 "R" V 5666 6500 50  0000 C CNN
-F 2 "" V 5480 6500 50  0001 C CNN
+F 2 "Resistors_SMD:R_0805" V 5480 6500 50  0001 C CNN
 F 3 "" H 5550 6500 50  0001 C CNN
 	1    5550 6500
@@
 F 0 "R4H1" V 5757 6850 50  0000 C CNN
 F 1 "R" V 5666 6850 50  0000 C CNN
-F 2 "" V 5480 6850 50  0001 C CNN
+F 2 "Resistors_SMD:R_0805" V 5480 6850 50  0001 C CNN
 F 3 "" H 5550 6850 50  0001 C CNN
 	1    5550 6850
@@
 F 0 "J1" H 3280 2042 50  0000 L CNN
 F 1 "Conn_01x08" H 3280 1951 50  0000 L CNN
-F 2 "" H 3200 2050 50  0001 C CNN
+F 2 "Pin_Headers:Pin_Header_Straight_1x08_Pitch2.54mm" H 3200 2050 50  0001 C CNN
 F 3 "" H 3200 2050 50  0001 C CNN
 	1    3200 2050
@@
 Text GLabel 3000 2150 0    60   Input ~ 0
 ~E
-Text GLabel 2800 2250 0    60   Input ~ 0
+Text GLabel 3000 2450 0    60   Input ~ 0
 S0
 Text GLabel 3000 2350 0    60   Input ~ 0
 S1
-Text GLabel 3000 2450 0    60   Input ~ 0
+Text GLabel 2850 2250 0    60   Input ~ 0
 S2
 $Comp
@@
 F 0 "J2" H 3280 2842 50  0000 L CNN
 F 1 "Screw_Terminal_01x02" H 3280 2751 50  0000 L CNN
-F 2 "" H 3200 2850 50  0001 C CNN
+F 2 "Connectors_Terminal_Blocks:TerminalBlock_4UCON_19963_02x3.5mm_Straight" H 3200 2850 50  0001 C CNN
 F 3 "" H 3200 2850 50  0001 C CNN
 	1    3200 2850
 	1    0    0    -1
 $EndComp
+Text GLabel 3000 2950 0    60   Input ~ 0
+PROBE_A
 Text GLabel 3000 2850 0    60   Input ~ 0
-PROBE_A
-Text GLabel 3000 2950 0    60   Input ~ 0
 PROBE_B
 $Comp
@@
 F 0 "U1" H 1775 4887 60  0000 C CNN
 F 1 "TLE2426" H 1775 4781 60  0000 C CNN
-F 2 "" H 1650 3800 60  0001 C CNN
+F 2 "SMD_Packages:SOIC-8-N" H 1650 3800 60  0001 C CNN
 F 3 "" H 1650 3800 60  0001 C CNN
 	1    1750 4350
@@
 F 0 "C1" V 2448 4100 50  0000 C CNN
 F 1 "C" V 2539 4100 50  0000 C CNN
-F 2 "" H 2738 3950 50  0001 C CNN
+F 2 "Capacitors_SMD:C_0805" H 2738 3950 50  0001 C CNN
 F 3 "" H 2700 4100 50  0001 C CNN
 	1    2700 4100
@@
 F 0 "C2" H 1685 5404 50  0000 R CNN
 F 1 "C" H 1685 5495 50  0000 R CNN
-F 2 "" H 1838 5300 50  0001 C CNN
+F 2 "Capacitors_SMD:C_0805" H 1838 5300 50  0001 C CNN
 F 3 "" H 1800 5450 50  0001 C CNN
 	1    1800 5450
@@
 F 0 "J3" V 6073 4730 50  0000 L CNN
 F 1 "Conn_01x02" V 6164 4730 50  0000 L CNN
-F 2 "" H 6200 4650 50  0001 C CNN
+F 2 "Pin_Headers:Pin_Header_Straight_1x02_Pitch2.54mm" H 6200 4650 50  0001 C CNN
 F 3 "" H 6200 4650 50  0001 C CNN
 	1    6200 4650
 	0    1    1    0
 $EndComp
+Text GLabel 4800 1850 0    60   Input ~ 0
+PROBE_A
+Text GLabel 4800 1950 0    60   Input ~ 0
+PROBE_B
+Text GLabel 4800 2050 0    60   Input ~ 0
+V_B
+Text GLabel 4800 2150 0    60   Input ~ 0
+V_C
+Text GLabel 4800 2250 0    60   Input ~ 0
+SIG_OUT
 Text GLabel 4800 1750 0    60   Input ~ 0
-PROBE_A
-Text GLabel 4800 1850 0    60   Input ~ 0
-PROBE_B
+SIG_IN
+$Comp
+L Conn_01x07 J4
+U 1 1 59CF2A95
+P 5000 2050
+F 0 "J4" H 5080 2092 50  0000 L CNN
+F 1 "Conn_01x07" H 5080 2001 50  0000 L CNN
+F 2 "Pin_Headers:Pin_Header_Straight_1x07_Pitch2.54mm" H 5000 2050 50  0001 C CNN
+F 3 "" H 5000 2050 50  0001 C CNN
+	1    5000 2050
+	1    0    0    -1
+$EndComp
+$Comp
+L GNDREF #PWR027
+U 1 1 59CF2D5A
+P 4800 2350
+F 0 "#PWR027" H 4800 2100 50  0001 C CNN
+F 1 "GNDREF" V 4805 2222 50  0000 R CNN
+F 2 "" H 4800 2350 50  0001 C CNN
+F 3 "" H 4800 2350 50  0001 C CNN
+	1    4800 2350
+	0    1    1    0
+$EndComp
 Wire Wire Line
 	6300 3200 6850 3200
 Wire Wire Line
-	6400 2900 6850 2900
-Wire Wire Line
-	6850 2900 6850 3050
-Wire Wire Line
-	6650 2900 6650 2500
-Connection ~ 6650 2900
+	6850 2500 6850 3050
 Wire Wire Line
 	5850 3200 6000 3200
@@
 	6200 3950 6200 4450
 Connection ~ 6200 3950
-Text GLabel 4800 2050 0    60   Input ~ 0
+Wire Wire Line
+	2800 2050 3000 2050
+Wire Wire Line
+	2850 2250 3000 2250
+Wire Wire Line
+	6850 3950 6850 4750
+Wire Wire Line
+	6850 4750 7050 4750
+Text GLabel 7050 4750 2    60   Input ~ 0
 V_B
-Text GLabel 4800 2150 0    60   Input ~ 0
+Wire Wire Line
+	7850 3950 7900 3950
+Text GLabel 7900 3950 2    60   Input ~ 0
 V_C
-$Comp
-L Conn_01x06 J4
-U 1 1 59CEEC19
-P 5000 1950
-F 0 "J4" H 5080 1942 50  0000 L CNN
-F 1 "Conn_01x06" H 5080 1851 50  0000 L CNN
-F 2 "" H 5000 1950 50  0001 C CNN
-F 3 "" H 5000 1950 50  0001 C CNN
-	1    5000 1950
-	1    0    0    -1
-$EndComp
-Text GLabel 4800 2250 0    60   Input ~ 0
-SIG_OUT
-Text GLabel 4800 1950 0    60   Input ~ 0
-SIG_IN
-Wire Wire Line
-	3000 2250 2800 2250
-Wire Wire Line
-	2800 2050 3000 2050
+Wire Wire Line
+	6550 2900 6450 2900
+Wire Wire Line
+	6450 2900 6450 3200
+Connection ~ 6450 3200
+Wire Wire Line
+	6850 2500 6650 2500
+Connection ~ 6850 2900
 $EndSCHEMATC

Commit message: update
Connections:
- net V_D: now reaches R10.1, R9.1, U3.14 (OUT_D)
- net V_D: now also J4.5 (Pin_5)
- net V_C: no longer names the net of D1.1 (K), D2.2 (A), U3.8 (OUT_C)
- net V_C: no longer J4.5 (Pin_5)
Changed lines of the file:
@@
 V_B
 Text GLabel 4800 2150 0    60   Input ~ 0
-V_C
+V_D
 Text GLabel 4800 2250 0    60   Input ~ 0
 SIG_OUT
@@
 Text GLabel 7050 4750 2    60   Input ~ 0
 V_B
-Text GLabel 7900 3950 2    60   Input ~ 0
-V_C
 Connection ~ 6850 2900
 Wire Wire Line
@@
 Wire Wire Line
 	6550 2900 6450 2900
-Wire Wire Line
-	7850 3950 7900 3950
 Wire Wire Line
 	6850 4750 7050 4750
@@
 Wire Wire Line
 	6300 3200 6850 3200
+Wire Wire Line
+	8050 2700 7950 2700
+Connection ~ 8050 2700
+Text GLabel 7950 2700 0    60   Input ~ 0
+V_D
 $EndSCHEMATC

Commit message: update
Parts:
- added J5, J6: Conn_Coaxial, Connectors:SMA_SMD_Jack_Straight, symbol Conn_Coaxial
- added J7, J9: Conn_01x04, Pin_Headers:Pin_Header_Straight_1x04_Pitch2.54mm, symbol Conn_01x04
Connections:
- net GND: now also J7.2 (Pin_2), J7.4 (Pin_4)
- net PROBE_A: now also J7.1 (Pin_1)
- net PROBE_B: now also J7.3 (Pin_3)
- new net: J5.1 (In), J9.2 (Pin_2)
- new net: J5.2 (Ext), J9.1 (Pin_1)
- new net: J6.1 (In), J9.4 (Pin_4)
- new net: J6.2 (Ext), J9.3 (Pin_3)
Changed lines of the file:
@@
 Text GLabel 7950 2700 0    60   Input ~ 0
 V_D
+$Comp
+L Conn_Coaxial J5
+U 1 1 59D3DE2D
+P 5800 1150
+F 0 "J5" H 5900 1034 50  0000 L CNN
+F 1 "Conn_Coaxial" H 5900 1125 50  0000 L CNN
+F 2 "Connectors:SMA_SMD_Jack_Straight" H 5800 1150 50  0001 C CNN
+F 3 "" H 5800 1150 50  0001 C CNN
+	1    5800 1150
+	-1   0    0    1
+$EndComp
+$Comp
+L Conn_Coaxial J6
+U 1 1 59D403CC
+P 6150 1450
+F 0 "J6" H 6250 1334 50  0000 L CNN
+F 1 "Conn_Coaxial" H 6250 1425 50  0000 L CNN
+F 2 "Connectors:SMA_SMD_Jack_Straight" H 6150 1450 50  0001 C CNN
+F 3 "" H 6150 1450 50  0001 C CNN
+	1    6150 1450
+	-1   0    0    1
+$EndComp
+$Comp
+L Conn_01x04 J9
+U 1 1 59D40983
+P 6650 1150
+F 0 "J9" H 6730 1142 50  0000 L CNN
+F 1 "Conn_01x04" H 6730 1051 50  0000 L CNN
+F 2 "Pin_Headers:Pin_Header_Straight_1x04_Pitch2.54mm" H 6650 1150 50  0001 C CNN
+F 3 "" H 6650 1150 50  0001 C CNN
+	1    6650 1150
+	1    0    0    -1
+$EndComp
+Wire Wire Line
+	5800 950  6450 950
+Wire Wire Line
+	6450 950  6450 1050
+Wire Wire Line
+	5950 1150 6450 1150
+Wire Wire Line
+	6150 1250 6450 1250
+Wire Wire Line
+	6300 1450 6450 1450
+Wire Wire Line
+	6450 1450 6450 1350
+Text GLabel 7950 1150 0    60   Input ~ 0
+PROBE_A
+Text GLabel 7950 1350 0    60   Input ~ 0
+PROBE_B
+$Comp
+L Conn_01x04 J7
+U 1 1 59D4C6FF
+P 8150 1250
+F 0 "J7" H 8230 1242 50  0000 L CNN
+F 1 "Conn_01x04" H 8230 1151 50  0000 L CNN
+F 2 "Pin_Headers:Pin_Header_Straight_1x04_Pitch2.54mm" H 8150 1250 50  0001 C CNN
+F 3 "" H 8150 1250 50  0001 C CNN
+	1    8150 1250
+	1    0    0    -1
+$EndComp
+$Comp
+L GND #PWR028
+U 1 1 59D4C787
+P 7950 1250
+F 0 "#PWR028" H 7950 1000 50  0001 C CNN
+F 1 "GND" V 7955 1122 50  0000 R CNN
+F 2 "" H 7950 1250 50  0001 C CNN
+F 3 "" H 7950 1250 50  0001 C CNN
+	1    7950 1250
+	0    1    1    0
+$EndComp
+$Comp
+L GND #PWR029
+U 1 1 59D4C7D4
+P 7950 1450
+F 0 "#PWR029" H 7950 1200 50  0001 C CNN
+F 1 "GND" V 7955 1322 50  0000 R CNN
+F 2 "" H 7950 1450 50  0001 C CNN
+F 3 "" H 7950 1450 50  0001 C CNN
+	1    7950 1450
+	0    1    1    0
+$EndComp
 $EndSCHEMATC
