File: conductive/conductive.kicad_pcb (KiCad board)
At the start: 2 copper layers, 59.1 x 40 mm, 29 parts, among them J1 Conn_01x08, J2 Screw_Terminal_01x02, J3 Conn_01x02, J4 Conn_01x07, U1 TLE2426, U2 74H4051, U3 AD8534, U4 AD8531

Commit message: update
Parts:
- moved J2 3.24 mm to (79.4, 61.0)
Routing:
- net +3V3: track 22.8 -> 52.6 mm, vias 2 -> 4
- net PROBE_B: track 75.3 -> 69.4 mm
- net GND: track 126.5 -> 124.2 mm

Commit message: update
Connections:
- D1 pad 1: V_C -> Net-(D1-Pad1)
- D2 pad 2: V_C -> Net-(D1-Pad1)
- J4 pad 5: V_C -> V_D
- R10 pad 1: Net-(R10-Pad1) -> V_D
- R9 pad 1: Net-(R10-Pad1) -> V_D
- U3 pad 14: Net-(R10-Pad1) -> V_D
- U3 pad 8: V_C -> Net-(D1-Pad1)
Routing:
- net V_D: track 0.00 -> 42.6 mm, vias 0 -> 4
- net V_C: track 26.4 -> 0.00 mm, vias 2 -> 0
- net Net-(D1-Pad1): track 0.00 -> 18.6 mm, vias 0 -> 2
- net Net-(R10-Pad1): track 16.5 -> 0.00 mm, vias 2 -> 0
- net PROBE_B: track 69.4 -> 71.1 mm

Commit message: update
Other:
- board text added: "3V3"
- board text added: "GND"
- board text added: "IN"
- board text added: "OUT"
- board text added: "PA"
- board text added: "PB"
- board text added: "R4"
- board text added: "S0"
- board text added: "S1"
- board text added: "S2"
- board text added: "VB"
- board text added: "VD"
- board text added: "VG"
- board text added: "~E"
Changed lines of the file:
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@@
   (general
     (thickness 1.6)
-    (drawings 6)
+    (drawings 24)
     (tracks 367)
     (zones 0)
@@
     )
   )
+  (gr_text PB (at 73.66 60.96) (layer F.SilkS)
+    (effects (font (size 1.5 1.5) (thickness 0.3)))
+  )
+  (gr_text PA (at 73.66 57.404) (layer F.SilkS)
+    (effects (font (size 1.5 1.5) (thickness 0.3)))
+  )
+  (gr_text R4 (at 43.688 80.518) (layer F.SilkS)
+    (effects (font (size 1.5 1.5) (thickness 0.3)))
+  )
+  (gr_text VG (at 71.882 79.756 90) (layer F.SilkS)
+    (effects (font (size 1.5 1.5) (thickness 0.3)))
+  )
+  (gr_text OUT (at 69.342 79.248 90) (layer F.SilkS)
+    (effects (font (size 1.5 1.5) (thickness 0.3)))
+  )
+  (gr_text VD (at 66.548 79.756 90) (layer F.SilkS)
+    (effects (font (size 1.5 1.5) (thickness 0.3)))
+  )
+  (gr_text VB (at 64.262 79.756 90) (layer F.SilkS)
+    (effects (font (size 1.5 1.5) (thickness 0.3)))
+  )
+  (gr_text PB (at 61.722 80.01 90) (layer F.SilkS)
+    (effects (font (size 1.5 1.5) (thickness 0.3)))
+  )
+  (gr_text PA (at 58.928 80.01 90) (layer F.SilkS)
+    (effects (font (size 1.5 1.5) (thickness 0.3)))
+  )
+  (gr_text IN (at 56.642 80.264 90) (layer F.SilkS)
+    (effects (font (size 1.5 1.5) (thickness 0.3)))
+  )
+  (gr_text S0 (at 31.496 70.104) (layer F.SilkS)
+    (effects (font (size 1.5 1.5) (thickness 0.3)))
+  )
+  (gr_text S1 (at 31.496 67.564) (layer F.SilkS)
+    (effects (font (size 1.5 1.5) (thickness 0.3)))
+  )
+  (gr_text S2 (at 31.496 64.77) (layer F.SilkS)
+    (effects (font (size 1.5 1.5) (thickness 0.3)))
+  )
+  (gr_text ~E (at 30.734 62.484) (layer F.SilkS)
+    (effects (font (size 1.5 1.5) (thickness 0.3)))
+  )
+  (gr_text OUT (at 32.004 59.69) (layer F.SilkS)
+    (effects (font (size 1.5 1.5) (thickness 0.3)))
+  )
+  (gr_text IN (at 30.988 57.15) (layer F.SilkS)
+    (effects (font (size 1.5 1.5) (thickness 0.3)))
+  )
+  (gr_text GND (at 32.004 54.61) (layer F.SilkS)
+    (effects (font (size 1.5 1.5) (thickness 0.3)))
+  )
+  (gr_text 3V3 (at 32.004 52.07) (layer F.SilkS)
+    (effects (font (size 1.5 1.5) (thickness 0.3)))
+  )
   (dimension 59.055 (width 0.3) (layer Dwgs.User)

Commit message: update
Parts:
- added J5: Conn_Coaxial, Connectors:SMA_SMD_Jack_Straight, F.Cu at (84.7, 61.8)
- added J6: Conn_Coaxial, Connectors:SMA_SMD_Jack_Straight, F.Cu at (84.7, 70.5)
- added J7: Conn_01x04, Pin_Headers:Pin_Header_Straight_1x04_Pitch2.54mm, F.Cu at (82.4, 77.3)
- added J9: Conn_01x04, Pin_Headers:Pin_Header_Straight_1x04_Pitch2.54mm, F.Cu at (85.0, 85.0)
- moved J2 8.20 mm to (84.7, 54.7)
- moved D2 6.69 mm to (74.4, 78.2)
- moved R8 5.27 mm to (75.4, 65.8)
- moved D1 4.67 mm to (74.4, 73.2)
- moved R7 4.33 mm to (70.4, 75.9)
- moved R6 2.26 mm to (75.4, 69.1)
- moved R9 2.20 mm to (75.4, 62.6)
Routing:
- net Net-(J5-Pad2): track 0.00 -> 38.2 mm, vias 0 -> 1
- net PROBE_B: track 71.1 -> 101.9 mm
- net PROBE_A: track 47.6 -> 78.1 mm
- net Net-(J5-Pad1): track 0.00 -> 24.8 mm, vias 0 -> 1
- net Net-(J6-Pad2): track 0.00 -> 17.8 mm
- net Net-(J6-Pad1): track 0.00 -> 9.77 mm, vias 0 -> 1
- net Net-(D1-Pad1): track 18.6 -> 9.17 mm, vias 2 -> 0
- net Net-(D2-Pad1): track 24.6 -> 15.6 mm
- net Net-(D1-Pad2): track 11.3 -> 6.71 mm
- net Net-(R8-Pad1): track 14.0 -> 10.0 mm
- net V_D: track 42.6 -> 39.8 mm
- net Net-(R5-Pad2): track 19.9 -> 18.6 mm
Other:
- board size 59.1 x 40 mm -> 66.7 x 41.9 mm
- board text added: "1"
- board text added: "2"
- board text added: "3"
- board text added: "4"

Commit message: update
Parts:
- added REF**: 1pin, Connectors:1pin, F.Cu at (29.0, 84.3)
- added REF**: 1pin, Connectors:1pin, F.Cu at (29.0, 51.8)
- moved J1 6.86 mm to (27.9, 58.9)
Routing:
- net S2: track 35.0 -> 27.4 mm
- net S1: track 38.3 -> 31.3 mm
- net S0: track 40.4 -> 34.3 mm
- net SIG_OUT: track 96.0 -> 98.9 mm
- net +3V3: track 52.1 -> 55.0 mm
- net ~E: track 23.9 -> 21.1 mm, vias 2 -> 1
- net SIG_IN: track 50.9 -> 52.2 mm
- net GND: track 124.2 -> 124.5 mm, vias 8 -> 7
