File: conductive/hbc_1.kicad_pcb (KiCad board)
At the start: 2 copper layers, 61 x 25.9 mm, 28 parts, among them J1 Conn_01x08, J2 Screw_Terminal_01x02, J3 Conn_01x02, U1 TLE2426, U2 74H4051, U3 AD8534, U4 AD8531

Commit message: update
Routing:
- net Net-(D1-Pad1): track 11.9 -> 15.4 mm
Other:
- board text added: "edgecollective.io/honeybear"
- board text added: "honeybear::conductivity"
Changed lines of the file:
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@@
   (general
     (thickness 1.6)
-    (drawings 16)
-    (tracks 382)
+    (drawings 17)
+    (tracks 383)
     (zones 0)
     (modules 28)
@@
     (pad_to_mask_clearance 0.2)
     (aux_axis_origin 0 0)
-    (grid_origin 86.36 77.724)
+    (grid_origin 22.352 89.916)
     (visible_elements FFFDFF7F)
     (pcbplotparams
@@
     (tags "capacitor 0805")
     (attr smd)
-    (fp_text reference C1 (at 0 -1.5 90) (layer F.SilkS)
+    (fp_text reference C1 (at 2.54 0 180) (layer F.SilkS)
       (effects (font (size 1 1) (thickness 0.15)))
     )
@@
       (effects (font (size 1 1) (thickness 0.15)))
     )
-    (fp_text user %R (at 0 -1.5 90) (layer F.Fab)
+    (fp_text user %R (at 2.54 0 180) (layer F.Fab)
       (effects (font (size 1 1) (thickness 0.15)))
     )
@@
     (tags "resistor 0805")
     (attr smd)
-    (fp_text reference R4B1 (at 0 -1.524 180) (layer F.SilkS)
+    (fp_text reference R4B1 (at -3.556 -1.016 180) (layer F.SilkS)
       (effects (font (size 1 1) (thickness 0.15)))
     )
@@
     (tags "resistor 0805")
     (attr smd)
-    (fp_text reference R4E1 (at 0 1.524 180) (layer F.SilkS)
+    (fp_text reference R4E1 (at 0 1.778 180) (layer F.SilkS)
       (effects (font (size 1 1) (thickness 0.15)))
     )
@@
     (tags "resistor 0805")
     (attr smd)
-    (fp_text reference R6 (at 0.762 1.778 180) (layer F.SilkS)
+    (fp_text reference R6 (at 0 2.032 180) (layer F.SilkS)
       (effects (font (size 1 1) (thickness 0.15)))
     )
@@
     (tags "resistor 0805")
     (attr smd)
-    (fp_text reference R7 (at 2.286 0.508 180) (layer F.SilkS)
+    (fp_text reference R7 (at 2.286 0.254 180) (layer F.SilkS)
       (effects (font (size 1 1) (thickness 0.15)))
     )
@@
     (tags "resistor 0805")
     (attr smd)
-    (fp_text reference R8 (at -2.54 1.016) (layer F.SilkS)
+    (fp_text reference R8 (at -2.54 0) (layer F.SilkS)
       (effects (font (size 1 1) (thickness 0.15)))
     )
@@
     )
   )
-  (dimension 29.972 (width 0.3) (layer Dwgs.User)
-    (gr_text "29.972 mm" (at 106.6965 73.914 90) (layer Dwgs.User)
-      (effects (font (size 1.5 1.5) (thickness 0.3)))
-    )
-    (feature1 (pts (xy 91.3765 58.928) (xy 108.0465 58.928)))
-    (feature2 (pts (xy 91.3765 88.9) (xy 108.0465 88.9)))
-    (crossbar (pts (xy 105.3465 88.9) (xy 105.3465 58.928)))
-    (arrow1a (pts (xy 105.3465 58.928) (xy 105.932921 60.054504)))
-    (arrow1b (pts (xy 105.3465 58.928) (xy 104.760079 60.054504)))
-    (arrow2a (pts (xy 105.3465 88.9) (xy 105.932921 87.773496)))
-    (arrow2b (pts (xy 105.3465 88.9) (xy 104.760079 87.773496)))
+  (gr_text edgecollective.io/honeybear (at 45.5295 68.961) (layer B.SilkS)
+    (effects (font (size 1.5 1.5) (thickness 0.3)) (justify mirror))
+  )
+  (gr_text honeybear::conductivity (at 48.0695 66.548) (layer B.SilkS)
+    (effects (font (size 1.5 1.5) (thickness 0.3)) (justify mirror))
   )
   (gr_line (start 83.312 64.008) (end 83.312 89.916) (angle 90) (layer Edge.Cuts) (width 0.15))
@@
     (effects (font (size 1.5 1.5) (thickness 0.3)))
   )
-  (gr_text S0 (at 29.6545 86.741) (layer F.SilkS)
+  (gr_text S2 (at 29.6545 86.741) (layer F.SilkS)
     (effects (font (size 1.5 1.5) (thickness 0.3)))
   )
@@
     (effects (font (size 1.5 1.5) (thickness 0.3)))
   )
-  (gr_text S2 (at 29.6545 81.407) (layer F.SilkS)
+  (gr_text S0 (at 29.6545 81.407) (layer F.SilkS)
     (effects (font (size 1.5 1.5) (thickness 0.3)))
   )
@@
   (segment (start 74.93 68.072) (end 73.914 67.056) (width 0.25) (layer F.Cu) (net 27))
   (segment (start 77.724 68.072) (end 74.93 68.072) (width 0.25) (layer F.Cu) (net 27))
+  (segment (start 66.572 86.106) (end 66.572 82.55) (width 0.25) (layer F.Cu) (net 28) (status C00000))
   (segment (start 66.572 83.058) (end 66.548 83.058) (width 0.25) (layer F.Cu) (net 28) (status C00000))
   (segment (start 66.548 83.058) (end 63.5 82.042) (width 0.25) (layer F.Cu) (net 28))
